File: Lambda_Project/KiCad/Steam_Controller/Steam_Controller.kicad_sch (KiCad schematic)
At the start: 156 parts, among them J1 MICROQTJ, P1 Conn_ARM_SWD_TagConnect_TC2030, P2 Conn_ARM_SWD_TagConnect_TC2030, P3 781271220, P4 781271220, Q10 DMN2300U-7, Q11 DMN2300U-7, Q12 DMP2035U-7, Q2 DMP2035U-7, Q3 MMBT3906, Q4 DMP2035U-7, Q5 DMP2035U-7, Q6 FDV304P, Q8 FDV304P, U1 LPC11U37FBD64/501,, U10 DMN63D8LDW-7, U2 TPD4E1U06DBVR - NG4P USB, U3 TPS61029DRCR, U4 TLV70230DBVT, U5 NRF51822-QFAB-T, U6 MPU6500, U7 A1304ELHLT-T, U8 A1304ELHLT-T, U9 DMN63D8LDW-7, X1 ABM8-12.000MHZ-B2-T, X2 NX2520SA-16MHZ-STD-CSW-5

Commit message: Fixed Models - Updated Values
Parts:
- R18: value 75kΩ -> 27kΩ
- X1: value ABM8-12.000MHZ-B2-T -> ABM8G-12.000MHZ-18-D2Y-T
Other:
- note removed: "*C8 and C9 might be 10pF caps. But I measured 18pF which is very odd."
Changed lines of the file:
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@@
 		)
 	)
-	(text "*C8 and C9 might be 10pF caps. But I measured 18pF which is very odd."
-		(exclude_from_sim no)
-		(at 318.262 42.672 0)
-		(effects
-			(font
-				(size 1.27 1.27)
-			)
-		)
-	)
 	(text "TODO: Sanity Check, reference datasheets, measure unsure values again."
 		(exclude_from_sim no)
@@
 		)
 	)
-	(label "* Double Check R18"
-		(at 204.47 367.03 180)
-		(effects
-			(font
-				(size 1.27 1.27)
-			)
-			(justify right bottom)
-		)
-	)
 	(label "* Double Check R26"
 		(at 215.9 325.12 0)
@@
 		)
 	)
-	(label "* Double check R42"
-		(at 170.18 391.16 0)
-		(effects
-			(font
-				(size 1.27 1.27)
-			)
-			(justify left bottom)
-		)
-	)
-	(label "* Double check C26, Capacitor went to space so using datasheet value for now"
-		(at 124.46 134.62 0)
-		(effects
-			(font
-				(size 1.27 1.27)
-			)
-			(justify left bottom)
-		)
-	)
 	(global_label "LB"
 		(shape input)
@@
 		(dnp no)
 		(property "Reference" "R18"
-			(at 188.468 372.364 90)
+			(at 189.738 363.982 90)
 			(effects
 				(font
@@
 			)
 		)
-		(property "Value" "75kΩ"
-			(at 189.23 370.078 90)
+		(property "Value" "27kΩ"
+			(at 191.008 366.268 90)
 			(effects
 				(font
@@
 			)
 		)
-		(property "Value" "ABM8-12.000MHZ-B2-T"
+		(property "Value" "ABM8G-12.000MHZ-18-D2Y-T"
 			(at 198.12 110.49 0)
 			(effects
