File: Lambda_Project/KiCad/Steam_Controller/Steam_Controller.kicad_pcb (KiCad board)
At the start: 2 copper layers, 151 x 77.4 mm, 214 parts, among them J1 MICROQTJ, P1 Conn_ARM_SWD_TagConnect_TC2030, P2 Conn_ARM_SWD_TagConnect_TC2030, P3 781271220, P4 781271220, Q10 DMN2300U-7, Q11 DMN2300U-7, Q12 DMP2035U-7, Q2 DMP2035U-7, Q3 MMBT3906, Q4 DMP2035U-7, Q5 DMP2035U-7, Q6 FDV304P, Q8 FDV304P, U1 LPC11U37FBD64/501,, U10 DMN63D8LDW-7, U2 TPD4E1U06DBVR - NG4P USB, U3 TPS61029DRCR, U4 TLV70230DBVT, U5 NRF51822-QFAB-T, U6 MPU6500, U7 A1304ELHLT-T, U8 A1304ELHLT-T, U9 DMN63D8LDW-7, X1 ABM8-12.000MHZ-B2-T, X2 NX2520SA-16MHZ-STD-CSW-5

Commit message: V1.0 Gerber files and cleanup
Routing:
- net HAL-VCC: track 154.1 -> 153.2 mm
Other:
- board text added: "Lambda_mainboard_EXP V1.0"
- board text removed: "Lambda_mainboard_EXP V0.99"
