File: Project_Janus/KiCad/Steam_Controller/Steam_Controller.kicad_sch (KiCad schematic)
At the start: 208 parts, among them IC1 nRF52833-QDAA-R, J1 MICROQTJ, P1 Conn_ARM_SWD_TagConnect_TC2030, P2 Conn_ARM_SWD_TagConnect_TC2030, P3 781271220, P4 781271220, Q10 DMN2300U-7, Q11 DMN2300U-7, Q12 DMP2035U-7, Q2 DMP2035U-7, Q3 MMBT3906, Q4 DMP2035U-7, Q5 DMP2035U-7, Q6 FDV304P, Q8 FDV304P, U10 DMN63D8LDW-7, U2 TPD4E1U06DBVR - NG4P USB, U3 TPS61029DRCR, U4 TLV70230DBVT, U5 NRF51822-QFAB-T, U6 MPU6500, U7 A1304ELHLT-T, U8 A1304ELHLT-T, U9 DMN63D8LDW-7, X1 ABM8-12.000MHZ-B2-T, X2 NX2520SA-16MHZ-STD-CSW-5

Commit message: nRF52833 Setup KiCad
Parts:
- added C10: 100pF, symbol Device:C
- added C11, C9: 100nF, symbol Device:C
- added C3: 1.0pF, symbol Device:C
- added C4: 1.2pF, symbol Device:C
- added C8: 820pF, symbol Device:C
- added L1: 4.7nH, symbol Device:L
- added L2: 2.2nH, symbol Device:L
Connections:
- net at IC1.21 (DEC5): now also C8.1
- net at IC1.24 (ANT): now also C3.1, L1.1
- net at IC1.26 (DEC6): now also IC1.38 (DEC4), C9.1
- net at IC1.27 (DEC3): now also C10.1
- net at IC1.30 (VDD_3): now also C11.1
- new net: C4.1, L1.2, L2.1
- new net GNDREF: C10.2, C11.2, C3.2, C4.2, C8.2, C9.2
- no-connect marks 0 -> 1
Other:
- moved on the sheet: BAT1, BAT2, C12, C13, C14, C15, C16, C17, C18, C19, C20, C22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
